File: schematics/UniversalSaftSwitch.sch (EAGLE design)
At the start: 20 parts, among them IC2 MAX485 CSA, IC3 AT90S2313S, K2 HF115F-024-S3, T1 BC817

Commit message: New Schematic
Signed-off-by: Ralf Ramsauer <ralf@ramses-pyramidenbau.de>
Parts:
- added C5, C6: 22p, rcl:C-EUC0805K
- added JP3: (no value), pinhead:PINHD-1X2
- added Q1: 14.2, crystal:CRYSTALHC49U-V
- added R4, R6: 0, rcl:R-EU_M0805
Connections:
- new net LED: IC3.(AIN0)PB0, R6.2
- new net N$10: C6.2, IC3.XTAL1, Q1.1
- new net N$11: JP2.1, R4.1
- new net N$12: JP3.1, R6.1
- new net N$7: C5.2, IC3.XTAL2, Q1.2
- net D+: now also IC2G$1.A, X1-4.KL; no longer IC2G$1.B, X1-3.KL
- net D-: now also IC2G$1.B, X1-3.KL; no longer IC2G$1.A, X1-4.KL
- net DE: no longer IC2G$1.RE/
- net GND: now also C5.1, C6.1, IC2G$1.RE/, JP3.2
- net PROG: now also R4.2; no longer JP2.1
Other:
- moved on the sheet: C1, C2, C3, C4, D2, IC2, IC2P, IC3, JP1, JP2, K2, LED1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

Commit message: New schematic + pcb
Signed-off-by: Ralf Ramsauer <ralf@ramses-pyramidenbau.de>
Parts:
- added R7: 0, rcl:R-EU_M0805
Connections:
- net GND: now also R7.1, R7.2
Changed lines of the file:
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@@
 <part name="R6" library="rcl" deviceset="R-EU_" device="M0805" value="0"/>
 <part name="R3" library="rcl" deviceset="R-EU_" device="M0805" value="0"/>
+<part name="R7" library="rcl" deviceset="R-EU_" device="M0805" value="0"/>
+<part name="GND11" library="supply1" deviceset="GND" device=""/>
+<part name="GND12" library="supply1" deviceset="GND" device=""/>
 </parts>
 <sheets>
@@
 <instance part="R6" gate="G$1" x="139.7" y="139.7" rot="R180"/>
 <instance part="R3" gate="G$1" x="200.66" y="144.78" rot="R180"/>
+<instance part="R7" gate="G$1" x="190.5" y="96.52" rot="R180"/>
+<instance part="GND11" gate="1" x="182.88" y="91.44"/>
+<instance part="GND12" gate="1" x="198.12" y="91.44"/>
 </instances>
 <busses>
@@
 <wire x1="147.32" y1="137.16" x2="147.32" y2="134.62" width="0.1524" layer="91"/>
 </segment>
+<segment>
+<pinref part="GND11" gate="1" pin="GND"/>
+<pinref part="R7" gate="G$1" pin="2"/>
+<wire x1="182.88" y1="93.98" x2="182.88" y2="96.52" width="0.1524" layer="91"/>
+<wire x1="182.88" y1="96.52" x2="185.42" y2="96.52" width="0.1524" layer="91"/>
+</segment>
+<segment>
+<pinref part="R7" gate="G$1" pin="1"/>
+<pinref part="GND12" gate="1" pin="GND"/>
+<wire x1="195.58" y1="96.52" x2="198.12" y2="96.52" width="0.1524" layer="91"/>
+<wire x1="198.12" y1="96.52" x2="198.12" y2="93.98" width="0.1524" layer="91"/>
+</segment>
 </net>
